File: hardware/EuroPi/kicad/europi.kicad_pcb (KiCad board)
At the start: 2 copper layers, 139.1 x 128.5 mm, 104 parts, among them IC1 TL074, IC2 TL074, IC3 MCP6002, J1 Thonkiconn_Mono_Jack, J2 Thonkiconn_Mono_Jack, J3 Thonkiconn_Mono_Jack, J4 Thonkiconn_Mono_Jack, J5 Thonkiconn_Mono_Jack, J6 Thonkiconn_Mono_Jack, J7 Thonkiconn_Mono_Jack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

Commit message: Fix OLED window offset, add OLED I2C labels
Other:
- outline, holes or cut-outs redrawn
- board text added: "GND"
- board text added: "SCL"
- board text added: "SDA"
- board text added: "VCC"
- board text added: "X"

Commit message: Remix v0.10.0-sss-tht production files
Parts:
- added CONN11: Conn_01x04_Counter_Clockwise_M, Connector_PinHeader_2.54mm:PinHeader_1x04_P2.54mm_Vertical, B.Cu at (8.71, 18.0)
- added JP1: SolderJumper_2_Bridged, Jumper:SolderJumper-2_P1.3mm_Bridged_Pad1.0x1.5mm, B.Cu at (6.06, 10.3)
- added JP2: SolderJumper_2_Bridged, Jumper:SolderJumper-2_P1.3mm_Bridged_Pad1.0x1.5mm, B.Cu at (6.06, 12.9)
- added JP3: SolderJumper_2_Bridged, Jumper:SolderJumper-2_P1.3mm_Bridged_Pad1.0x1.5mm, B.Cu at (6.06, 15.4)
- added JP4: SolderJumper_2_Bridged, Jumper:SolderJumper-2_P1.3mm_Bridged_Pad1.0x1.5mm, B.Cu at (6.06, 17.9)
Routing:
- net /+3.3V J: track 64.1 -> 70.2 mm
- net /OLED SDA J: track 15.6 -> 20.4 mm
- net Earth: track 583.2 -> 587.2 mm
- net /OLED SCL J: track 23.6 -> 22.3 mm
Other:
- board text removed: "GND"
- board text removed: "SCL"
- board text removed: "SDA"
- board text removed: "VCC"
- board text removed: "X"
