File: hardware/EuroPi/kicad/europi.kicad_sch (KiCad schematic)
At the start: 96 parts, among them IC1 TL074, IC2 TL074, IC3 MCP6002, J1 Thonkiconn_Mono_Jack, J2 Thonkiconn_Mono_Jack, J3 Thonkiconn_Mono_Jack, J4 Thonkiconn_Mono_Jack, J5 Thonkiconn_Mono_Jack, J6 Thonkiconn_Mono_Jack, J7 Thonkiconn_Mono_Jack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

Commit message: Remix v0.10.0-sss-tht production files
Parts:
- added CONN11: Conn_01x04_Counter_Clockwise_M, Connector_PinHeader_2.54mm:PinHeader_1x04_P2.54mm_Vertical, symbol Connector_Generic:Conn_01x04
- added JP1, JP2, JP3, JP4: SolderJumper_2_Bridged, Jumper:SolderJumper-2_P1.3mm_Bridged_Pad1.0x1.5mm, symbol Jumper:SolderJumper_2_Bridged
Connections:
- net +3.3V J: now also CONN11.2 (Pin_2), JP3.1 (A), JP3.2 (B)
- net Earth: now also CONN11.1 (Pin_1), JP4.1 (A), JP4.2 (B)
- net OLED SCL J: now also CONN11.3 (Pin_3), JP2.1 (A), JP2.2 (B)
- net OLED SDA J: now also CONN11.4 (Pin_4), JP1.1 (A), JP1.2 (B)
Changed lines of the file:
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@@
     (stroke (width 0) (type default))
   )
+  (wire (pts (xy 441.452 248.666) (xy 457.962 248.666))
+    (stroke (width 0) (type default))
+  )
   (wire (pts (xy 271.145 49.53) (xy 271.145 40.64))
     (stroke (width 0) (type default))
@@
     (stroke (width 0) (type default))
   )
+  (wire (pts (xy 465.582 248.666) (xy 482.092 248.666))
+    (stroke (width 0) (type default))
+  )
   (wire (pts (xy 80.645 250.19) (xy 84.455 250.19))
     (stroke (width 0) (type default))
@@
     (stroke (width 0) (type default))
   )
+  (wire (pts (xy 482.092 246.126) (xy 465.582 246.126))
+    (stroke (width 0) (type default))
+  )
   (polyline (pts (xy 309.88 199.39) (xy 309.88 144.78))
     (stroke (width 0) (type default))
   )
+  (wire (pts (xy 465.582 243.586) (xy 482.092 243.586))
+    (stroke (width 0) (type default))
+  )
   (wire (pts (xy 80.645 252.73) (xy 84.455 252.73))
     (stroke (width 0) (type default))
@@
     (stroke (width 0) (type default))
   )
+  (wire (pts (xy 465.582 251.206) (xy 482.092 251.206))
+    (stroke (width 0) (type default))
+  )
   (wire (pts (xy 60.96 121.92) (xy 73.66 121.92))
     (stroke (width 0) (type default))
@@
     (stroke (width 0) (type default))
   )
+  (wire (pts (xy 441.452 243.586) (xy 457.962 243.586))
+    (stroke (width 0) (type default))
+  )
   (polyline (pts (xy 360.553 246.126) (xy 397.383 246.126))
     (stroke (width 0) (type default))
@@
     (stroke (width 0) (type default))
   )
+  (wire (pts (xy 457.962 246.126) (xy 441.452 246.126))
+    (stroke (width 0) (type default))
+  )
   (wire (pts (xy 266.065 36.83) (xy 266.065 40.64))
     (stroke (width 0) (type default))
@@
     (stroke (width 0) (type default))
   )
+  (wire (pts (xy 441.452 251.206) (xy 457.962 251.206))
+    (stroke (width 0) (type default))
+  )
   (polyline (pts (xy 99.06 149.86) (xy 99.06 110.49))
     (stroke (width 0) (type default))
@@
     (effects (font (size 1.27 1.27)) (justify left bottom))
   )
+  (label "OLED SDA J" (at 467.741 243.586 0) (fields_autoplaced)
+    (effects (font (size 1.27 1.27)) (justify left bottom))
+  )
   (label "GP16" (at 309.88 38.1 0) (fields_autoplaced)
     (effects (font (size 1.27 1.27)) (justify left bottom))
@@
     (effects (font (size 1.27 1.27)) (justify left bottom))
   )
+  (label "+3.3V J" (at 451.358 248.666 180) (fields_autoplaced)
+    (effects (font (size 1.27 1.27)) (justify right bottom))
+  )
   (label "+3.3V J" (at 368.935 216.535 0) (fields_autoplaced)
     (effects (font (size 1.27 1.27)) (justify left bottom))
@@
     (effects (font (size 1.27 1.27)) (justify right bottom))
   )
+  (label "EARTH J" (at 451.739 251.206 180) (fields_autoplaced)
+    (effects (font (size 1.27 1.27)) (justify right bottom))
+  )
   (label "OUTPUT 3 P" (at 443.865 229.235 90) (fields_autoplaced)
     (effects (font (size 1.27 1.27)) (justify left bottom))
@@
     (effects (font (size 1.27 1.27)) (justify left bottom))
   )
+  (label "OLED SCL J" (at 443.738 246.126 0) (fields_autoplaced)
+    (effects (font (size 1.27 1.27)) (justify left bottom))
+  )
+  (label "OLED SCL J" (at 467.868 246.126 0) (fields_autoplaced)
+    (effects (font (size 1.27 1.27)) (justify left bottom))
+  )
   (label "GP15" (at 38.1 265.43 0) (fields_autoplaced)
     (effects (font (size 1.27 1.27)) (justify left bottom))
@@
     (effects (font (size 1.27 1.27)) (justify left bottom))
   )
+  (label "OLED SDA J" (at 443.611 243.586 0) (fields_autoplaced)
+    (effects (font (size 1.27 1.27)) (justify left bottom))
+  )
   (label "+5V" (at 100.965 217.17 0) (fields_autoplaced)
     (effects (font (size 1.27 1.27)) (justify left bottom))
@@
     (effects (font (size 1.27 1.27)) (justify right bottom))
   )
+  (label "EARTH J" (at 475.869 251.206 180) (fields_autoplaced)
+    (effects (font (size 1.27 1.27)) (justify right bottom))
+  )
   (label "+12V" (at 267.335 217.17 0) (fields_autoplaced)
     (effects (font (size 1.27 1.27)) (justify left bottom))
@@
     (effects (font (size 1.27 1.27)) (justify left bottom))
   )
+  (label "+3.3V J" (at 475.488 248.666 180) (fields_autoplaced)
+    (effects (font (size 1.27 1.27)) (justify right bottom))
+  )
   (label "OLED SDA J" (at 455.549 259.588 0) (fields_autoplaced)
     (effects (font (size 1.27 1.27)) (justify left bottom))
@@
     )
   )
+  (symbol (lib_id "Jumper:SolderJumper_2_Bridged") (at 461.772 246.126 0) (unit 1)
+    (in_bom yes) (on_board yes) (dnp no)
+    (property "Reference" "JP2" (at 465.836 244.094 0)
+      (effects (font (size 1.27 1.27)) hide)
+    )
+    (property "Value" "SolderJumper_2_Bridged" (at 461.772 243.332 0)
+      (effects (font (size 1.27 1.27)) hide)
+    )
+    (property "Footprint" "Jumper:SolderJumper-2_P1.3mm_Bridged_Pad1.0x1.5mm" (at 461.772 246.126 0)
+      (effects (font (size 1.27 1.27)) hide)
+    )
+    (property "Datasheet" "~" (at 461.772 246.126 0)
+      (effects (font (size 1.27 1.27)) hide)
+    )
+    (pin "1")
+    (pin "2")
+    (instances
+      (project "europi"
+        (path "/a8447faf-e0a0-4c4a-ae53-4d4b28669151"
+          (reference "JP2") (unit 1)
+        )
+      )
+    )
+  )
   (symbol (lib_id "Amplifier_Operational:TL074") (at 350.52 96.52 0) (unit 4)
     (in_bom yes) (on_board yes) (dnp no) (fields_autoplaced)
@@
     )
   )
+  (symbol (lib_id "Jumper:SolderJumper_2_Bridged") (at 461.772 243.586 0) (unit 1)
+    (in_bom yes) (on_board yes) (dnp no)
+    (property "Reference" "JP1" (at 461.772 238.252 0)
+      (effects (font (size 1.27 1.27)) hide)
+    )
+    (property "Value" "SolderJumper_2_Bridged" (at 462.026 238.252 0)
+      (effects (font (size 1.27 1.27)))
+    )
+    (property "Footprint" "Jumper:SolderJumper-2_P1.3mm_Bridged_Pad1.0x1.5mm" (at 461.772 243.586 0)
+      (effects (font (size 1.27 1.27)) hide)
+    )
+    (property "Datasheet" "~" (at 461.772 243.586 0)
+      (effects (font (size 1.27 1.27)) hide)
+    )
+    (pin "1")
+    (pin "2")
+    (instances
+      (project "europi"
+        (path "/a8447faf-e0a0-4c4a-ae53-4d4b28669151"
+          (reference "JP1") (unit 1)
+        )
+      )
+    )
+  )
   (symbol (lib_id "Eurorack:Thonkiconn_Mono_Jack") (at 331.47 170.18 0) (unit 1)
     (in_bom yes) (on_board yes) (dnp no) (fields_autoplaced)
@@
     )
   )
+  (symbol (lib_id "Jumper:SolderJumper_2_Bridged") (at 461.772 248.666 0) (unit 1)
+    (in_bom yes) (on_board yes) (dnp no) (fields_autoplaced)
+    (property "Reference" "JP3" (at 461.772 245.364 0)
+      (effects (font (size 1.27 1.27)) hide)
+    )
+    (property "Value" "SolderJumper_2_Bridged" (at 461.772 245.872 0)
+      (effects (font (size 1.27 1.27)) hide)
+    )
+    (property "Footprint" "Jumper:SolderJumper-2_P1.3mm_Bridged_Pad1.0x1.5mm" (at 461.772 248.666 0)
+      (effects (font (size 1.27 1.27)) hide)
+    )
+    (property "Datasheet" "~" (at 461.772 248.666 0)
+      (effects (font (size 1.27 1.27)) hide)
+    )
+    (pin "1")
+    (pin "2")
+    (instances
+      (project "europi"
+        (path "/a8447faf-e0a0-4c4a-ae53-4d4b28669151"
+          (reference "JP3") (unit 1)
+        )
+      )
+    )
+  )
   (symbol (lib_id "power:Earth") (at 113.665 238.76 0) (unit 1)
     (in_bom yes) (on_board yes) (dnp no)
@@
     )
   )
+  (symbol (lib_id "Connector_Generic:Conn_01x04") (at 436.372 248.666 180) (unit 1)
+    (in_bom yes) (on_board yes) (dnp no) (fields_autoplaced)
+    (property "Reference" "CONN11" (at 436.372 237.49 0)
+      (effects (font (size 1.27 1.27)))
+    )
+    (property "Value" "Conn_01x04_Counter_Clockwise_M" (at 436.372 240.03 0)
+      (effects (font (size 1.27 1.27)))
+    )
+    (property "Footprint" "Connector_PinHeader_2.54mm:PinHeader_1x04_P2.54mm_Vertical" (at 436.372 248.666 0)
+      (effects (font (size 1.27 1.27)) hide)
+    )
+    (property "Datasheet" "~" (at 436.372 248.666 0)
+      (effects (font (size 1.27 1.27)) hide)
+    )
+    (pin "1")
+    (pin "2")
+    (pin "3")
+    (pin "4")
+    (instances
+      (project "europi"
+        (path "/a8447faf-e0a0-4c4a-ae53-4d4b28669151"
+          (reference "CONN11") (unit 1)
+        )
+      )
+    )
+  )
   (symbol (lib_id "Eurorack:Thonkiconn_Mono_Jack") (at 197.485 91.44 0) (mirror y) (unit 1)
     (in_bom yes) (on_board yes) (dnp no) (fields_autoplaced)
@@
         )
       )
+    )
+  )
+  (symbol (lib_id "Jumper:SolderJumper_2_Bridged") (at 461.772 251.206 0) (unit 1)
+    (in_bom yes) (on_board yes) (dnp no)
+    (property "Reference" "JP4" (at 473.456 251.714 0)
+      (effects (font (size 1.27 1.27)) hide)
+    )
+    (property "Value" "SolderJumper_2_Bridged" (at 466.09 254 0)
+      (effects (font (size 1.27 1.27)) hide)
+    )
+    (property "Footprint" "Jumper:SolderJumper-2_P1.3mm_Bridged_Pad1.0x1.5mm" (at 461.772 251.206 0)
+      (effects (font (size 1.27 1.27)) hide)
+    )
+    (property "Datasheet" "~" (at 461.772 251.206 0)
+      (effects (font (size 1.27 1.27)) hide)
+    )
+    (pin "1")
+    (pin "2")
+    (instances
+      (project "europi"
+        (path "/a8447faf-e0a0-4c4a-ae53-4d4b28669151"
+          (reference "JP4") (unit 1)
+        )
+      )
